File: hardware/controller.kicad_sch (KiCad schematic)
At the start: 61 parts, among them J11 UART, J12 JST 2.0 BATT, J9 Chip Enable, P1 USB_C_Plug_USB2.0, U1 THB001P, U5 ESP32-H2-MINI-1, U6 AP2204, U7 MCP73833

Commit message: hardware v1.0
Parts:
- removed C14: 2.2uF, Capacitor_SMD:C_0603_1608Metric, symbol SAMC21_breakout-rescue:C
- removed C15: 10uF, Capacitor_SMD:C_0603_1608Metric, symbol SAMC21_breakout-rescue:C
- removed C16: 10uF, Capacitor_SMD:C_0603_1608Metric, symbol Device:C
- removed C17: 22uF, Capacitor_SMD:C_0603_1608Metric, symbol Device:C
- removed D1, D8, D9: LED, Capacitor_SMD:C_0603_1608Metric, symbol SAMC21_breakout-rescue:LED-RESCUE-SAMC21_breakout
- removed D5: TPD1E10B06DPYR, Diode_SMD:D_SOD-523, symbol custom_IC:TPD1E10B06DPYR
- removed D6: PWLED, Diode_SMD:D_0603_1608Metric, symbol Device:LED
- removed J11: UART, Connector_PinHeader_2.54mm:PinHeader_1x04_P2.54mm_Vertical, symbol Connector:Conn_01x04_Male
- removed J12: JST 2.0 BATT, Connector_JST:JST_PH_B2B-PH-K_1x02_P2.00mm_Vertical, symbol Connector_Generic:Conn_01x02
- removed J9: Chip Enable, Connector_PinHeader_2.54mm:PinHeader_1x02_P2.54mm_Vertical, symbol Connector:Conn_01x02_Male
- removed R1, R12, R13, R25: 200, Resistor_SMD:R_0603_1608Metric, symbol SAMC21_breakout-rescue:R
- removed R16: 1M, Resistor_SMD:R_0603_1608Metric, symbol Device:R
- removed R17, R18: 5k1, Resistor_SMD:R_0603_1608Metric, symbol Device:R
- removed R20, R21: 470, Resistor_SMD:R_0603_1608Metric, symbol Device:R
- removed R22, R23: 1.43K, Resistor_SMD:R_0603_1608Metric, symbol Device:R
- removed R24: 75K, Resistor_SMD:R_0603_1608Metric, symbol Device:R
- removed S4: TL4100AF240QG_, kicad_reformed_custom_IC:SW_PTS810_SJM_250_SMTR_LFS, symbol custom_IC:TL4100AF240QG_
- removed TP1: 0_IN1, TestPoint:TestPoint_Pad_1.0x1.0mm, symbol Connector:TestPoint
- removed TP2: 0_IN2, TestPoint:TestPoint_Pad_1.0x1.0mm, symbol Connector:TestPoint
- removed U6: AP2204, kicad_reformed_custom_IC:AP2204, symbol SAMC21_breakout-rescue:AP2204
- removed U7: MCP73833, kicad_reformed_custom_IC:SON50P300X300X100-11N, symbol custom_IC:MCP73833
- added C1, C2, C3, C4: 10uF, Capacitor_SMD:C_0603_1608Metric, symbol Device:C
- added C10, C11, C12: 0.1uF, Capacitor_SMD:C_0603_1608Metric, symbol Device:C
- added C20: 1uF, Capacitor_SMD:C_0603_1608Metric, symbol Device:C
- added C5: 47uF, Capacitor_SMD:C_0603_1608Metric, symbol Device:C
- added C6, C7: 10uF, Capacitor_SMD:C_0603_1608Metric, symbol SAMC21_breakout-rescue:C
- added D1: TPD1E10B06DPYR, Diode_SMD:D_SOD-523, symbol custom_IC:TPD1E10B06DPYR
- added J1: JST 2.0 BATT, Connector_JST:JST_PH_S2B-PH-SM4-TB_1x02-1MP_P2.00mm_Horizontal, symbol Connector_Generic:Conn_01x02
- added L1: 1uH, custom_IC:RES_CIGT252010, symbol Device:L
- added LED1, LED2, LED3: IN-PI15TAT5R5G5B, custom_IC:IN-PI15_INL, symbol custom_IC:IN-PI15TAT5R5G5B
- added Q1: BSS138, Package_TO_SOT_SMD:SOT-23, symbol Transistor_FET:BSS138
- added R1: 806, Resistor_SMD:R_0603_1608Metric, symbol Device:R
- added R11: 330, Resistor_SMD:R_0603_1608Metric, symbol Device:R
- added R12, R13, R14, R27, R6: 10K, Resistor_SMD:R_0603_1608Metric, symbol Device:R
- added R15: 470, Resistor_SMD:R_0603_1608Metric, symbol Device:R
- added R2: 1.43K, Resistor_SMD:R_0603_1608Metric, symbol Device:R
- added R26: 100K, Resistor_SMD:R_0603_1608Metric, symbol Device:R
- added R3: 91, Resistor_SMD:R_0603_1608Metric, symbol Device:R
- added R4: 75K, Resistor_SMD:R_0603_1608Metric, symbol Device:R
- added R5, R7, R8: 5K1, Resistor_SMD:R_0603_1608Metric, symbol Device:R
- added R9: 1M, Resistor_SMD:R_0603_1608Metric, symbol Device:R
- added S6: TL4100AF240QG_, kicad_reformed_custom_IC:SW_PTS810_SJM_250_SMTR_LFS, symbol custom_IC:TL4100AF240QG_
- added TP3, TP5: TP, TestPoint:TestPoint_Pad_1.5x1.5mm, symbol Connector:TestPoint
- added U1: AP2205, kicad_reformed_custom_IC:AP2204, symbol SAMC21_breakout-rescue:AP2204
- added U2: TPS631000DRLR, custom_IC:TPS631000DRLR_TEX, symbol custom_IC:TPS631000DRLR
- added U3: MCP73833, kicad_reformed_custom_IC:SON50P300X300X100-11N, symbol custom_IC:MCP73833
- C14: renamed from C10; value 1uF 25V -> 1uF
- C16: renamed from C1; value 1uF 25V -> 1uF
- C17: renamed from C2; value 1uF 25V -> 1uF
- C18: renamed from C3; value 1uF 25V -> 1uF
- C19: renamed from C4; value 1uF 25V -> 1uF
- D2: value LED -> LED_GREEN
- D3: value LED -> LED_RED
- R10: value 10k -> 330
- R16: renamed from R11; value 10k -> 10K
- R17: renamed from R9; value 10k -> 10K
- R18: renamed from R2; value 10k -> 10K
- R19: renamed from R4; value 10k -> 10K
- R20: renamed from R6; value 10k -> 10K
- R21: renamed from R8; value 10k -> 10K
- R22: renamed from R3; value 100k -> 100K
- R23: renamed from R5; value 100k -> 100K
- R24: renamed from R7; value 100k -> 100K
- R25: renamed from R14; value 100k -> 100K
- TH1: value TH 10k -> TH 10K
- TP1: renamed from TP3; footprint TestPoint:TestPoint_Pad_D1.0mm -> TestPoint:TestPoint_Pad_1.5x1.5mm
- renumbered C12 to C15, C9 to C8, C11 to C9, S5 to S4, S6 to S5, U5 to U4, U1 to U5
Connections:
- net +3V3: now also U5.B, C7.1, Q1.1 (G), R13.2, U1.5 (VOUT); no longer U5.C
- net +5V: now also C1.1, C10.1, C11.1, C12.1, C2.1, C6.1, LED1.2 (VDD), LED2.2 (VDD), LED3.2 (VDD), R1.1, R14.2, U1.1 (VIN), U1.3 (EN), U2.1 (VOUT); no longer P1.A4 (VBUS), P1.A9 (VBUS), P1.B4 (VBUS), P1.B9 (VBUS)
- net ADC_BATT: now also U4.19 (IO5), R12.2; no longer R10.2, U4.5 (IO2)
- net CHRGR+: now also C5.1, U3.10 (VBAT), U3.9 (VBAT)
- net GND: now also C1.2, C10.2, C11.2, C12.2, C2.2, C20.2, C3.2, C4.2, C5.2, C6.2, C7.2, D1.2, J1.1 (Pin_1), LED1.4 (GND), LED2.4 (GND), LED3.4 (GND), R26.2, R3.2, R4.1, R5.2, R6.1, R7.2, R8.2, R9.2, S6.1, U1.2 (GND), U2.7 (GND), U3.11 (PAD), U3.5 (VSS); no longer D2.1 (K), D3.1 (K)
- net LIPO+: now also J1.2 (Pin_2), R12.1; no longer R10.1
- net SW_A: now also U4.12 (IO13); no longer U4.19 (IO5)
- net SW_B: now also U4.13 (IO14); no longer U4.20 (IO10)
- net VR_BTN: now also R27.2
- net at U4.23 (IO9): now also S6.2
- net at U4.25 (IO25): now also Q1.2 (S), R13.1
- net USB_D-: now reaches U4.26 (IO26)
- net USB_D-: now also P1.A7 (D-)
- net USB_D+: now reaches U4.27 (IO27)
- net USB_D+: now also P1.A6 (D+)
- net at P1.S1 (SHIELD): now also R9.1
- net at D3.2 (A): now also R11.2
- net at P1.B5 (VCONN): now also R7.1
- net at TH1.1: now also R2.1, R4.2
- net at D2.2 (A): now also R10.2
- net at P1.A5 (CC): now also R8.1
- net U0RXD: no longer names the net of U4.30 (RXD0)
- net U0TXD: no longer names the net of U4.31 (TXD0)
- net raw_voltage renamed RAW
- net RAW: now also C3.1, U2.4 (VIN), U2.5 (EN)
- new net: R6.2, U2.6 (MODE)
- new net: TP5.1, U4.20 (IO10)
- new net: TP3.1, U4.5 (IO2)
- new net: R1.2, R3.1, U2.8 (FB)
- new net: LED1.3 (DOUT), LED2.1 (DIN)
- new net: LED2.3 (DOUT), LED3.1 (DIN)
- new net: R5.1, U3.6 (PROG)
- new net: R2.2, U3.8 (THERM)
- new net: C20.1, R26.1, R27.1
- new net: L1.1, U2.3 (LX1)
- new net: L1.2, U2.2 (LX2)
- new net: LED1.1 (DIN), R15.2
- new net: Q1.3 (D), R14.1, R15.1
- new net +5VD: C4.1, D1.1, P1.A4 (VBUS), P1.A9 (VBUS), P1.B4 (VBUS), P1.B9 (VBUS), R10.1, R11.1, U3.1 (VDD), U3.2 (VDD)
- new net STAT1_CHARGING: D3.1 (K), U3.3 (STAT1)
- new net STAT2_DONE: D2.1 (K), U3.4 (STAT2)
- no-connect marks 14 -> 15
Other:
- note added: "5V"
- note added: "Buttons"
- note added: "Charging"
- note added: "Done"
- note added: "Lets the USB controller know we want to charge"
- note added: "Lights"
- note added: "Lipo voltage is between 2.7V and 4.2V"
- note added: "Place close to U3"
- note added: "Power"
- note added: "Transistor for logic level shift"
- note added: "Using LEDs for charge status"
- note removed: "Connection Status"
- note removed: "GREEN LED"
- note removed: "Misc"
- note removed: "Power Status"
- note removed: "RED LED"
- note removed: "Signals to MCU indicating state of charge"
- note removed: "USB C Power Only"
- note removed: "USB4105-GF-A"
- note removed: "replace with 10K?"
- company: StuckAtPrototype -> StuckAtPrototype LLC
- moved on the sheet: C13, C14, C15, C16, C17, C18, C19, C8, C9, R16, R17, R18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
